Commit message: organization

File: simulation_ws/src/m2wr_description/urdf/m2wr.xacro (robot description, xacro)
@@ -26,5 +26,5 @@
       <material name="blue"/>
     </visual>
-    <!-- caster front -->
+    <!-- caster front-->
     <collision name="caster_front_collision">
       <origin rpy=" 0 0 0" xyz="0.35 0 -0.05"/>
@@ -48,5 +48,5 @@
         <sphere radius="0.05"/>
       </geometry>
-    </visual>
+    </visual>>
   </link>
   <link name="sensor_laser">
@@ -104,6 +104,6 @@
     </joint>
   <xacro:link_wheel name="link_right_wheel" />
-  <xacro:joint_wheel name="joint_right_wheel" child="link_right_wheel" origin_xyz="-0.05 0.20 0" />
+  <xacro:joint_wheel name="joint_right_wheel" child="link_right_wheel" origin_xyz="-0.05 0.18 0" />
   <xacro:link_wheel name="link_left_wheel" />
-  <xacro:joint_wheel name="joint_left_wheel" child="link_left_wheel" origin_xyz="-0.05 -0.20 0" />
+  <xacro:joint_wheel name="joint_left_wheel" child="link_left_wheel" origin_xyz="-0.05 -0.18 0" />
 </robot>

File: simulation_ws/src/m2wr_description/urdf/macros.xacro (robot description, xacro)
@@ -6,5 +6,6 @@
               <mass value="0.2"/>
               <origin rpy="0 1.5707 1.5707" xyz="0 0 0"/>
-              <inertia ixx="0.000526666666667" ixy="0" ixz="0" iyy="0.000526666666667" iyz="0" izz="0.001"/>
+              <!--inertia ixx="0.000526666666667" ixy="0" ixz="0" iyy="0.000526666666667" iyz="0" izz="0.001"/-->
+              <xacro:cylinder_inertia mass="0.2" r="0.1" l="0.04" />
             </inertial>
             <collision name="link_right_wheel_collision">
